Commit message: Contains updated code with option for gui controller, but gui controller joints are not aligned; not going to fix that

File: urdf/bittle_static.urdf (robot description, URDF)
Before this commit: robot bittle, 13 links, 12 joints
Links:
- link left-front-knee-link: geometry collision mesh filename=package://quad_walk/obj/left_knee.003c.obj scale=1.0 1.0 1.0; visual mesh filename=package://quad_walk/obj/left_knee.obj scale=1.0 1.0 1.0
- link right-back-knee-link: geometry collision mesh filename=package://quad_walk/obj/right_knee.002c.obj scale=1.0 1.0 1.0; visual mesh filename=package://quad_walk/obj/right_knee.001.obj scale=1.0 1.0 1.0
- link right-front-knee-link: geometry collision mesh filename=package://quad_walk/obj/right_knee.003c.obj scale=1.0 1.0 1.0; visual mesh filename=package://quad_walk/obj/right_knee.obj scale=1.0 1.0 1.0

Commit message: wrote basic code to get quad to stand up; currently does a barrel roll on rising; looking to change controller to effort based rather than position based

File: urdf/bittle_static.urdf (robot description, URDF)
Before this commit: robot bittle, 13 links, 12 joints
Joints:
- joint left_back_knee_joint: limit lower=-1.22173 upper=1.48353 effort=1.0 velocity=1.5708 -> lower=-1.22173 upper=1.48353 effort=0.5 velocity=1.5708
- joint left_back_shoulder_joint: limit lower=-1.5708 upper=1.22173 effort=1.0 velocity=1.5708 -> lower=-1.5708 upper=1.22173 effort=0.5 velocity=1.5708
- joint left_front_knee_joint: limit lower=-1.22173 upper=1.48353 effort=1.0 velocity=1.5708 -> lower=-1.22173 upper=1.48353 effort=0.5 velocity=1.5708
- joint left_front_shoulder_joint: limit lower=-1.5708 upper=1.22173 effort=1.0 velocity=1.5708 -> lower=-1.5708 upper=1.22173 effort=0.5 velocity=1.5708
- joint right_back_knee_joint: limit lower=-1.22173 upper=1.48353 effort=1.0 velocity=1.5708 -> lower=-1.22173 upper=1.48353 effort=0.5 velocity=1.5708
- joint right_back_shoulder_joint: limit lower=-1.5708 upper=1.22173 effort=1.0 velocity=1.5708 -> lower=-1.5708 upper=1.22173 effort=0.5 velocity=1.5708
- joint right_front_knee_joint: limit lower=-1.22173 upper=1.48353 effort=1.0 velocity=1.5708 -> lower=-1.22173 upper=1.48353 effort=0.5 velocity=1.5708
- joint right_front_shoulder_joint: limit lower=-1.5708 upper=1.22173 effort=1.0 velocity=1.5708 -> lower=-1.5708 upper=1.22173 effort=0.5 velocity=1.5708
