Commit message: Effort controller set up; need to tune pid gains; effort set at 2 for joints, results in jittery motion; need to look into programming joint state trajectory controller

File: urdf/bittle.urdf (robot description, URDF)
Before this commit: robot bittle, 13 links, 12 joints
Links:
- link left-front-knee-link: geometry collision mesh filename=package://quad_walk/obj/left_knee.003c.obj scale=1.0 1.0 1.0; visual mesh filename=package://quad_walk/obj/left_knee.obj scale=1.0 1.0 1.0
- link right-back-knee-link: geometry collision mesh filename=package://quad_walk/obj/right_knee.002c.obj scale=1.0 1.0 1.0; visual mesh filename=package://quad_walk/obj/right_knee.001.obj scale=1.0 1.0 1.0
- link right-front-knee-link: geometry collision mesh filename=package://quad_walk/obj/right_knee.003c.obj scale=1.0 1.0 1.0; visual mesh filename=package://quad_walk/obj/right_knee.obj scale=1.0 1.0 1.0
Joints:
- removed joint battery-joint
- removed joint cover-joint
- removed joint left-back-knee-joint
- removed joint left-back-shoulder-joint
- removed joint left-front-knee-joint
- removed joint left-front-shoulder-joint
- removed joint right-back-knee-joint
- removed joint right-back-shoulder-joint
- removed joint right-front-knee-joint
- removed joint right-front-shoulder-joint
- added joint battery_joint: type fixed, parent base-frame-link, child battery-link, origin xyz=0.00047 -0.00917 -0.04848 rpy=0 0 0
- added joint cover_joint: type fixed, parent base-frame-link, child cover-link, origin xyz=0.0014 0 0.1251 rpy=0 0 0
- added joint left_back_knee_joint: type revolute, parent left-back-shoulder-link, child left-back-knee-link, origin xyz=0 -0.49172 0 rpy=0 0 0, axis 0 0 1.0, limit lower=-1.22173 upper=1.48353 effort=2 velocity=1.5708
- added joint left_back_shoulder_joint: type revolute, parent base-frame-link, child left-back-shoulder-link, origin xyz=-0.44596 -0.51923 -0.02102 rpy=1.5708 0 -1.5708, axis 0 0 1.0, limit lower=-1.5708 upper=1.22173 effort=2 velocity=1.5708
- added joint left_front_knee_joint: type revolute, parent left-front-shoulder-link, child left-front-knee-link, origin xyz=6e-05 -0.49172 0 rpy=0 0 0, axis 0 0 1.0, limit lower=-1.22173 upper=1.48353 effort=2 velocity=1.5708
- added joint left_front_shoulder_joint: type revolute, parent base-frame-link, child left-front-shoulder-link, origin xyz=-0.44596 0.52264 -0.02102 rpy=1.5708 0 -1.5708, axis 0 0 1.0, limit lower=-1.5708 upper=1.22173 effort=2 velocity=1.5708
- added joint right_back_knee_joint: type revolute, parent right-back-shoulder-link, child right-back-knee-link, origin xyz=0.00015 0.49938 0.03996 rpy=0 0 3.14159, axis 0 0 1.0, limit lower=-1.22173 upper=1.48353 effort=2 velocity=1.5708
- added joint right_back_shoulder_joint: type revolute, parent base-frame-link, child right-back-shoulder-link, origin xyz=0.45149 -0.51923 -0.02102 rpy=-1.5708 0 -1.5708, axis 0 0 1.0, limit lower=-1.5708 upper=1.22173 effort=2 velocity=1.5708
- added joint right_front_knee_joint: type revolute, parent right-front-shoulder-link, child right-front-knee-link, origin xyz=6e-05 0.49938 0.03996 rpy=0 0 3.14159, axis 0 0 1.0, limit lower=-1.22173 upper=1.48353 effort=2 velocity=1.5708
- added joint right_front_shoulder_joint: type revolute, parent base-frame-link, child right-front-shoulder-link, origin xyz=0.45149 0.52264 -0.02102 rpy=-1.5708 0 -1.5708, axis 0 0 1.0, limit lower=-1.5708 upper=1.22173 effort=2 velocity=1.5708

Commit message: effort controller working; torque and pid values working; need to work on converting CoM trajectory to servo commands

File: urdf/bittle.urdf (robot description, URDF)
Before this commit: robot bittle, 13 links, 12 joints
Joints:
- joint left_back_knee_joint: limit lower=-1.22173 upper=1.48353 effort=2 velocity=1.5708 -> lower=-1.22173 upper=1.48353 effort=5 velocity=1.5708
- joint left_back_shoulder_joint: limit lower=-1.5708 upper=1.22173 effort=2 velocity=1.5708 -> lower=-1.5708 upper=1.22173 effort=5 velocity=1.5708
- joint left_front_knee_joint: limit lower=-1.22173 upper=1.48353 effort=2 velocity=1.5708 -> lower=-1.22173 upper=1.48353 effort=5 velocity=1.5708
- joint left_front_shoulder_joint: limit lower=-1.5708 upper=1.22173 effort=2 velocity=1.5708 -> lower=-1.5708 upper=1.22173 effort=5 velocity=1.5708
- joint right_back_knee_joint: limit lower=-1.22173 upper=1.48353 effort=2 velocity=1.5708 -> lower=-1.22173 upper=1.48353 effort=5 velocity=1.5708
- joint right_back_shoulder_joint: limit lower=-1.5708 upper=1.22173 effort=2 velocity=1.5708 -> lower=-1.5708 upper=1.22173 effort=5 velocity=1.5708
- joint right_front_knee_joint: limit lower=-1.22173 upper=1.48353 effort=2 velocity=1.5708 -> lower=-1.22173 upper=1.48353 effort=5 velocity=1.5708
- joint right_front_shoulder_joint: limit lower=-1.5708 upper=1.22173 effort=2 velocity=1.5708 -> lower=-1.5708 upper=1.22173 effort=5 velocity=1.5708

Commit message: effort controller updated with revolute accurate joint values; have knee and shoulder length values; need to start to convert trajectory to joint values

File: urdf/bittle.urdf (robot description, URDF)
Before this commit: robot bittle, 13 links, 12 joints
Joints:
- joint left_back_shoulder_joint: limit lower=-1.5708 upper=1.22173 effort=5 velocity=1.5708 -> lower=-1.22173 upper=1.22173 effort=5 velocity=1.5708
- joint right_back_knee_joint: limit lower=-1.22173 upper=1.48353 effort=5 velocity=1.5708 -> lower=-1.48353 upper=1.22173 effort=5 velocity=1.5708
- joint right_back_shoulder_joint: limit lower=-1.5708 upper=1.22173 effort=5 velocity=1.5708 -> lower=-1.22173 upper=1.22173 effort=5 velocity=1.5708
- joint right_front_knee_joint: limit lower=-1.22173 upper=1.48353 effort=5 velocity=1.5708 -> lower=-1.48353 upper=1.22173 effort=5 velocity=1.5708
- joint right_front_shoulder_joint: limit lower=-1.5708 upper=1.22173 effort=5 velocity=1.5708 -> lower=-1.22173 upper=1.5708 effort=5 velocity=1.5708

Commit message: notes in readme

File: urdf/bittle.urdf (robot description, URDF)
Before this commit: robot bittle, 13 links, 12 joints
Joints:
- joint left_back_knee_joint: limit lower=-1.22173 upper=1.48353 effort=5 velocity=1.5708 -> lower=-1.22173 upper=1.48353 effort=50 velocity=1.5708
- joint left_back_shoulder_joint: limit lower=-1.22173 upper=1.22173 effort=5 velocity=1.5708 -> lower=-1.22173 upper=1.22173 effort=50 velocity=1.5708
- joint left_front_knee_joint: limit lower=-1.22173 upper=1.48353 effort=5 velocity=1.5708 -> lower=-1.22173 upper=1.48353 effort=50 velocity=1.5708
- joint left_front_shoulder_joint: limit lower=-1.5708 upper=1.22173 effort=5 velocity=1.5708 -> lower=-1.5708 upper=1.22173 effort=50 velocity=1.5708
- joint right_back_knee_joint: limit lower=-1.48353 upper=1.22173 effort=5 velocity=1.5708 -> lower=-1.48353 upper=1.22173 effort=50 velocity=1.5708
- joint right_back_shoulder_joint: limit lower=-1.22173 upper=1.22173 effort=5 velocity=1.5708 -> lower=-1.22173 upper=1.22173 effort=50 velocity=1.5708
- joint right_front_knee_joint: limit lower=-1.48353 upper=1.22173 effort=5 velocity=1.5708 -> lower=-1.48353 upper=1.22173 effort=50 velocity=1.5708
- joint right_front_shoulder_joint: limit lower=-1.22173 upper=1.5708 effort=5 velocity=1.5708 -> lower=-1.22173 upper=1.5708 effort=50 velocity=1.5708

Commit message: working inverse kinematics, but copies every single vector right now; PID controllers for effort joints needs to be tuned, still jittery, causing instability in robot; next step is trajectory generation to step coordination

File: urdf/bittle.urdf (robot description, URDF)
Before this commit: robot bittle, 13 links, 12 joints
Joints:
- joint left_back_knee_joint: limit lower=-1.22173 upper=1.48353 effort=50 velocity=1.5708 -> lower=-1.22173 upper=1.48353 effort=10 velocity=1.5708
- joint left_back_shoulder_joint: limit lower=-1.22173 upper=1.22173 effort=50 velocity=1.5708 -> lower=-1.22173 upper=1.22173 effort=10 velocity=1.5708
- joint left_front_knee_joint: limit lower=-1.22173 upper=1.48353 effort=50 velocity=1.5708 -> lower=-1.22173 upper=1.48353 effort=10 velocity=1.5708
- joint left_front_shoulder_joint: limit lower=-1.5708 upper=1.22173 effort=50 velocity=1.5708 -> lower=-1.5708 upper=1.22173 effort=10 velocity=1.5708
- joint right_back_knee_joint: limit lower=-1.48353 upper=1.22173 effort=50 velocity=1.5708 -> lower=-1.48353 upper=1.22173 effort=10 velocity=1.5708
- joint right_back_shoulder_joint: limit lower=-1.22173 upper=1.22173 effort=50 velocity=1.5708 -> lower=-1.22173 upper=1.22173 effort=10 velocity=1.5708
- joint right_front_knee_joint: limit lower=-1.48353 upper=1.22173 effort=50 velocity=1.5708 -> lower=-1.48353 upper=1.22173 effort=10 velocity=1.5708
- joint right_front_shoulder_joint: limit lower=-1.22173 upper=1.5708 effort=50 velocity=1.5708 -> lower=-1.22173 upper=1.5708 effort=10 velocity=1.5708

Commit message: knees collision meshes are detailed cad models, which will result in better performance, but will have higher computational needs

File: urdf/bittle.urdf (robot description, URDF)
Before this commit: robot bittle, 13 links, 12 joints
Links:
- link left-back-knee-link: geometry collision mesh filename=package://quad_walk/obj/left_knee.001.obj scale=1.0 1.0 1.0; visual mesh filename=package://quad_walk/obj/left_knee.001.obj scale=1.0 1.0 1.0
- link left-front-knee-link: geometry collision mesh filename=package://quad_walk/obj/left_knee.obj scale=1.0 1.0 1.0; visual mesh filename=package://quad_walk/obj/left_knee.obj scale=1.0 1.0 1.0
- link right-back-knee-link: geometry collision mesh filename=package://quad_walk/obj/right_knee.001.obj scale=1.0 1.0 1.0; visual mesh filename=package://quad_walk/obj/right_knee.001.obj scale=1.0 1.0 1.0
- link right-front-knee-link: geometry collision mesh filename=package://quad_walk/obj/right_knee.obj scale=1.0 1.0 1.0; visual mesh filename=package://quad_walk/obj/right_knee.obj scale=1.0 1.0 1.0
